File: mochi_companion/GPS.kicad_sch (KiCad schematic)
At the start: 20 parts, among them J3 Conn_Coaxial, U7 AT2659, U8 MAX-M8C

Commit message: 250712_0041
Parts:
- removed C18: 470p, Capacitor_SMD:C_0201_0603Metric, symbol Device:C
- removed R13: 0R, Resistor_SMD:R_0201_0603Metric, symbol Device:R
- added C38: 100n, Capacitor_SMD:C_0402_1005Metric, symbol Device:C
- added R17: 10k, PCM_Resistor_SMD_AKL:R_0402_1005Metric, symbol Device:R
- C14: footprint Capacitor_SMD:C_0201_0603Metric -> Capacitor_SMD:C_0402_1005Metric; Field5 (none) -> C0402; Field6 (none) -> 50V
- C15: value 33p -> 470P; footprint Capacitor_SMD:C_0201_0603Metric -> Capacitor_SMD:C_0402_1005Metric; Field5 (none) -> C0402; Field6 (none) -> 50V; now fitted
- C16: value 100n -> 33p; footprint Capacitor_SMD:C_0201_0603Metric -> Capacitor_SMD:C_0402_1005Metric; Field5 (none) -> C0402; Field6 (none) -> 50V; now not fitted
- C17, C19, C20: value 4.7u -> 4u7; footprint Capacitor_SMD:C_0201_0603Metric -> Capacitor_SMD:C_0402_1005Metric; Field5 (none) -> C0402; Field6 (none) -> 16V
- D1, D2: footprint LED_SMD:LED_0201_0603Metric -> Diode_SMD:D_0402_1005Metric; Field5 (none) -> D0402
- J3: footprint (none) -> Connector_Coaxial:U.FL_Molex_MCRF_73412-0110_Vertical; now not fitted
- L3: footprint Capacitor_SMD:C_0201_0603Metric -> Inductor_SMD:L_0402_1005Metric; Field5 (none) -> L0402
- L4: footprint Inductor_SMD:L_0201_0603Metric -> Inductor_SMD:L_0402_1005Metric; Field5 (none) -> L0402
- L5: value 47n -> 6.8n; footprint Inductor_SMD:L_0201_0603Metric -> Inductor_SMD:L_0402_1005Metric; Field5 (none) -> L0402
- R12: value 1k -> 0R; footprint Resistor_SMD:R_0201_0603Metric -> PCM_Resistor_SMD_AKL:R_0402_1005Metric; Field5 (none) -> R0402; now not fitted
- R14: value 10k -> 1k; footprint Resistor_SMD:R_0201_0603Metric -> PCM_Resistor_SMD_AKL:R_0402_1005Metric; Field5 (none) -> R0402
Connections:
- net +3.3V: now also R12.2, C38.1, R17.2; no longer C16.1, R14.1
- net GND: now also C38.2; no longer C15.2
- net at L3.2, U7.6 (RF_OUT), U8.11 (RF_IN): now also C16.1, L5.1; no longer C15.1, L5.2
- net at C14.1, L3.1: now also J3.1 (In); no longer AE2.1 (A), AE3.1 (A)
- net at U8.14 (VCC_RF): now also L5.2; no longer L5.1
- net at R14.2: now also U8.4 (TIMEPULSE); no longer U8.9 (~{RESET})
- net at D1.1 (K), D2.2 (A): now also R14.1; no longer R12.2
- net at U8.7 (VCC_IO): now also R12.1
- net at L4.1: now also C15.2
- new net: AE2.1 (A), AE3.1 (A), C15.1
- new net: R17.1, U8.9 (~{RESET})

Commit message: 250713_0019
Parts:
- removed AE2: Antenna, PrjLib:antenna_pad, symbol Device:Antenna
- renumbered AE3 to AE1, C14 to C11, C15 to C12, C16 to C13, C38 to C14, C17 to C15, C19 to C16, C20 to C17, D1 to D3, D2 to D4, L3 to L1, L4 to L2, L5 to L3, R14 to R11, R17 to R13, U7 to U2, U8 to U3
Changed lines of the file:
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@@
-	)
-	(junction
-		(at 81.28 78.74)
-		(diameter 0)
-		(color 0 0 0 0)
 	)
 	(junction
@@
 	(wire
 		(pts
-			(xy 81.28 78.74) (xy 81.28 86.36)
-		)
-		(stroke
-			(width 0)
-			(type default)
-		)
-	)
-	(wire
-		(pts
 			(xy 132.08 69.85) (xy 132.08 86.36)
 		)
@@
 	(wire
 		(pts
-			(xy 69.85 77.47) (xy 69.85 78.74)
+			(xy 69.85 77.47) (xy 69.85 86.36)
 		)
 		(stroke
@@
 	(wire
 		(pts
-			(xy 81.28 77.47) (xy 81.28 78.74)
-		)
-		(stroke
-			(width 0)
-			(type default)
-		)
-	)
-	(wire
-		(pts
 			(xy 153.67 97.79) (xy 160.02 97.79)
 		)
@@
 	(wire
 		(pts
-			(xy 69.85 78.74) (xy 81.28 78.74)
-		)
-		(stroke
-			(width 0)
-			(type default)
-		)
-	)
-	(wire
-		(pts
-			(xy 81.28 86.36) (xy 83.82 86.36)
+			(xy 69.85 86.36) (xy 83.82 86.36)
 		)
 		(stroke
@@
 		(on_board yes)
 		(dnp no)
-		(property "Reference" "C38"
+		(property "Reference" "C14"
 			(at 145.288 74.422 0)
 			(effects
@@
 			(project "mochi_companios"
 				(path "/4ca1c142-b31d-4c3e-804c-2439f9285e87/c53c7e95-cdb8-4a5f-949f-3e233653d611"
-					(reference "C38")
+					(reference "C14")
 					(unit 1)
 				)
@@
 		(on_board yes)
 		(dnp yes)
-		(property "Reference" "C14"
+		(property "Reference" "C11"
 			(at 84.328 102.362 0)
 			(effects
@@
 			(project "mochi_companios"
 				(path "/4ca1c142-b31d-4c3e-804c-2439f9285e87/c53c7e95-cdb8-4a5f-949f-3e233653d611"
-					(reference "C14")
+					(reference "C11")
 					(unit 1)
 				)
@@
 		(on_board yes)
 		(dnp no)
-		(property "Reference" "#PWR028"
+		(property "Reference" "#PWR029"
 			(at 142.24 86.36 0)
 			(effects
@@
 			(project "mochi_companios"
 				(path "/4ca1c142-b31d-4c3e-804c-2439f9285e87/c53c7e95-cdb8-4a5f-949f-3e233653d611"
-					(reference "#PWR028")
+					(reference "#PWR029")
 					(unit 1)
 				)
@@
 		(on_board yes)
 		(dnp no)
-		(property "Reference" "R14"
+		(property "Reference" "R11"
 			(at 155.194 111.76 0)
 			(effects
@@
 			(project "mochi_companios"
 				(path "/4ca1c142-b31d-4c3e-804c-2439f9285e87/c53c7e95-cdb8-4a5f-949f-3e233653d611"
-					(reference "R14")
+					(reference "R11")
 					(unit 1)
 				)
@@
 		(dnp no)
 		(fields_autoplaced yes)
-		(property "Reference" "U7"
+		(property "Reference" "U2"
 			(at 121.285 78.74 0)
 			(effects
@@
 			)
 		)
-		(property "Description" " Low Noise Amplifiers (LNA) - RF"
+		(property "Description" "Low Noise Amplifiers (LNA) - RF"
 			(at 119.634 82.042 0)
 			(effects
@@
 			(project "mochi_companios"
 				(path "/4ca1c142-b31d-4c3e-804c-2439f9285e87/c53c7e95-cdb8-4a5f-949f-3e233653d611"
-					(reference "U7")
+					(reference "U2")
 					(unit 1)
 				)
@@
 		(on_board yes)
 		(dnp yes)
-		(property "Reference" "L3"
+		(property "Reference" "L1"
 			(at 85.852 93.726 90)
 			(effects
@@
 			(project "mochi_companios"
 				(path "/4ca1c142-b31d-4c3e-804c-2439f9285e87/c53c7e95-cdb8-4a5f-949f-3e233653d611"
-					(reference "L3")
+					(reference "L1")
 					(unit 1)
 				)
@@
 		(on_board yes)
 		(dnp no)
-		(property "Reference" "C17"
+		(property "Reference" "C15"
 			(at 215.138 74.422 0)
 			(effects
@@
 			(project "mochi_companios"
 				(path "/4ca1c142-b31d-4c3e-804c-2439f9285e87/c53c7e95-cdb8-4a5f-949f-3e233653d611"
-					(reference "C17")
+					(reference "C15")
 					(unit 1)
 				)
@@
 		(on_board yes)
 		(dnp yes)
-		(property "Reference" "D1"
+		(property "Reference" "D3"
 			(at 141.732 123.952 90)
 			(effects
@@
 			(project "mochi_companios"
 				(path "/4ca1c142-b31d-4c3e-804c-2439f9285e87/c53c7e95-cdb8-4a5f-949f-3e233653d611"
-					(reference "D1")
+					(reference "D3")
 					(unit 1)
 				)
@@
 		(on_board yes)
 		(dnp no)
-		(property "Reference" "C19"
+		(property "Reference" "C16"
 			(at 227.838 74.422 0)
 			(effects
@@
 			(project "mochi_companios"
 				(path "/4ca1c142-b31d-4c3e-804c-2439f9285e87/c53c7e95-cdb8-4a5f-949f-3e233653d611"
-					(reference "C19")
-					(unit 1)
-				)
-			)
-		)
-	)
-	(symbol
-		(lib_id "Device:Antenna")
-		(at 81.28 72.39 0)
-		(unit 1)
-		(exclude_from_sim no)
-		(in_bom yes)
-		(on_board yes)
-		(dnp no)
-		(fields_autoplaced yes)
-		(property "Reference" "AE2"
-			(at 83.82 71.755 0)
-			(effects
-				(font
-					(size 1.27 1.27)
-				)
-				(justify left)
-			)
-		)
-		(property "Value" "Antenna"
-			(at 83.82 74.295 0)
-			(effects
-				(font
-					(size 1.27 1.27)
-				)
-				(justify left)
-			)
-		)
-		(property "Footprint" "PrjLib:antenna_pad"
-			(at 81.28 72.39 0)
-			(effects
-				(font
-					(size 1.27 1.27)
-				)
-				(hide yes)
-			)
-		)
-		(property "Datasheet" "~"
-			(at 81.28 72.39 0)
-			(effects
-				(font
-					(size 1.27 1.27)
-				)
-				(hide yes)
-			)
-		)
-		(property "Description" ""
-			(at 81.28 72.39 0)
-			(effects
-				(font
-					(size 1.27 1.27)
-				)
-				(hide yes)
-			)
-		)
-		(pin "1"
-		)
-		(instances
-			(project "mochi_companios"
-				(path "/4ca1c142-b31d-4c3e-804c-2439f9285e87/c53c7e95-cdb8-4a5f-949f-3e233653d611"
-					(reference "AE2")
+					(reference "C16")
 					(unit 1)
 				)
@@
 		(on_board yes)
 		(dnp no)
-		(property "Reference" "C15"
+		(property "Reference" "C12"
 			(at 88.138 79.502 90)
 			(effects
@@
 			(project "mochi_companios"
 				(path "/4ca1c142-b31d-4c3e-804c-2439f9285e87/c53c7e95-cdb8-4a5f-949f-3e233653d611"
-					(reference "C15")
+					(reference "C12")
 					(unit 1)
 				)
@@
 		(on_board yes)
 		(dnp no)
-		(property "Reference" "L5"
+		(property "Reference" "L3"
 			(at 154.432 83.82 0)
 			(effects
@@
 			(project "mochi_companios"
 				(path "/4ca1c142-b31d-4c3e-804c-2439f9285e87/c53c7e95-cdb8-4a5f-949f-3e233653d611"
-					(reference "L5")
+					(reference "L3")
 					(unit 1)
 				)
@@
 		(on_board yes)
 		(dnp no)
-		(property "Reference" "R17"
+		(property "Reference" "R13"
 			(at 200.914 74.93 0)
 			(effects
@@
 			(project "mochi_companios"
 				(path "/4ca1c142-b31d-4c3e-804c-2439f9285e87/c53c7e95-cdb8-4a5f-949f-3e233653d611"
-					(reference "R17")
+					(reference "R13")
 					(unit 1)
 				)
@@
 		(on_board yes)
 		(dnp no)
-		(property "Reference" "C20"
+		(property "Reference" "C17"
 			(at 240.538 74.422 0)
 			(effects
@@
 			(project "mochi_companios"
 				(path "/4ca1c142-b31d-4c3e-804c-2439f9285e87/c53c7e95-cdb8-4a5f-949f-3e233653d611"
-					(reference "C20")
+					(reference "C17")
 					(unit 1)
 				)
@@
 		(on_board yes)
 		(dnp no)
-		(property "Reference" "#PWR031"
+		(property "Reference" "#PWR028"
 			(at 110.49 99.06 0)
 			(effects
@@
 			(project "mochi_companios"
 				(path "/4ca1c142-b31d-4c3e-804c-2439f9285e87/c53c7e95-cdb8-4a5f-949f-3e233653d611"
-					(reference "#PWR031")
+					(reference "#PWR028")
 					(unit 1)
 				)
@@
 		(on_board yes)
 		(dnp no)
-		(property "Reference" "#PWR030"
+		(property "Reference" "#PWR031"
 			(at 153.67 133.35 0)
 			(effects
@@
 			(project "mochi_companios"
 				(path "/4ca1c142-b31d-4c3e-804c-2439f9285e87/c53c7e95-cdb8-4a5f-949f-3e233653d611"
-					(reference "#PWR030")
+					(reference "#PWR031")
 					(unit 1)
 				)
@@
 		(on_board yes)
 		(dnp yes)
-		(property "Reference" "C16"
+		(property "Reference" "C13"
 			(at 97.028 102.362 0)
 			(effects
@@
 			(project "mochi_companios"
 				(path "/4ca1c142-b31d-4c3e-804c-2439f9285e87/c53c7e95-cdb8-4a5f-949f-3e233653d611"
-					(reference "C16")
+					(reference "C13")
 					(unit 1)
 				)
@@
 		(on_board yes)
 		(dnp no)
-		(property "Reference" "U8"
+		(property "Reference" "U3"
 			(at 180.34 114.3 0)
 			(effects
@@
 			(project "mochi_companios"
 				(path "/4ca1c142-b31d-4c3e-804c-2439f9285e87/c53c7e95-cdb8-4a5f-949f-3e233653d611"
-					(reference "U8")
+					(reference "U3")
 					(unit 1)
 				)
@@
 		(on_board yes)
 		(dnp no)
-		(property "Reference" "L4"
+		(property "Reference" "L2"
 			(at 93.472 82.296 90)
 			(effects
@@
 			(project "mochi_companios"
 				(path "/4ca1c142-b31d-4c3e-804c-2439f9285e87/c53c7e95-cdb8-4a5f-949f-3e233653d611"
-					(reference "L4")
+					(reference "L2")
 					(unit 1)
 				)
@@
 		(dnp no)
 		(fields_autoplaced yes)
-		(property "Reference" "AE3"
+		(property "Reference" "AE1"
 			(at 72.39 71.755 0)
 			(effects
@@
 			(project "mochi_companios"
 				(path "/4ca1c142-b31d-4c3e-804c-2439f9285e87/c53c7e95-cdb8-4a5f-949f-3e233653d611"
-					(reference "AE3")
+					(reference "AE1")
 					(unit 1)
 				)
@@
 		(on_board yes)
 		(dnp no)
-		(property "Reference" "D2"
+		(property "Reference" "D4"
 			(at 156.718 122.428 90)
 			(effects
@@
 			(project "mochi_companios"
 				(path "/4ca1c142-b31d-4c3e-804c-2439f9285e87/c53c7e95-cdb8-4a5f-949f-3e233653d611"
-					(reference "D2")
+					(reference "D4")
 					(unit 1)
 				)
@@
 		(on_board yes)
 		(dnp no)
-		(property "Reference" "#PWR037"
+		(property "Reference" "#PWR025"
 			(at 67.31 114.3 0)
 			(effects
@@
 			(project "mochi_companios"
 				(path "/4ca1c142-b31d-4c3e-804c-2439f9285e87/c53c7e95-cdb8-4a5f-949f-3e233653d611"
-					(reference "#PWR037")
+					(reference "#PWR025")
 					(unit 1)
 				)
@@
 		(on_board yes)
 		(dnp no)
-		(property "Reference" "#PWR029"
+		(property "Reference" "#PWR030"
 			(at 144.78 123.19 0)
 			(effects
@@
 			(project "mochi_companios"
 				(path "/4ca1c142-b31d-4c3e-804c-2439f9285e87/c53c7e95-cdb8-4a5f-949f-3e233653d611"
-					(reference "#PWR029")
-					(unit 1)
-				)
+					(reference "#PWR030")
+					(unit 1)
+				)
