File: mochi_companion/OLED.kicad_sch (KiCad schematic)
At the start: 13 parts

Commit message: 250713_0019
Parts:
- renumbered C55 to C47, C5 to C48, C23 to C49, C24 to C50, C64 to C51, C65 to C52, C66 to C53, D4 to D8, R106 to R40, R47 to R41, R46 to R42, R115 to R43
Changed lines of the file:
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@@
 		(on_board yes)
 		(dnp no)
-		(property "Reference" "#PWR0221"
+		(property "Reference" "#PWR0109"
 			(at 177.8 148.59 0)
 			(effects
@@
 			(project "mochi_companios"
 				(path "/4ca1c142-b31d-4c3e-804c-2439f9285e87/15ca05c3-044e-4926-b1a3-d57223b2942a"
-					(reference "#PWR0221")
+					(reference "#PWR0109")
 					(unit 1)
 				)
@@
 		(on_board yes)
 		(dnp no)
-		(property "Reference" "C65"
+		(property "Reference" "C52"
 			(at 201.168 54.102 0)
 			(effects
@@
 			(project "mochi_companios"
 				(path "/4ca1c142-b31d-4c3e-804c-2439f9285e87/15ca05c3-044e-4926-b1a3-d57223b2942a"
-					(reference "C65")
+					(reference "C52")
 					(unit 1)
 				)
@@
 		(on_board yes)
 		(dnp no)
-		(property "Reference" "#PWR0220"
+		(property "Reference" "#PWR0103"
 			(at 153.67 148.59 0)
 			(effects
@@
 			(project "mochi_companios"
 				(path "/4ca1c142-b31d-4c3e-804c-2439f9285e87/15ca05c3-044e-4926-b1a3-d57223b2942a"
-					(reference "#PWR0220")
+					(reference "#PWR0103")
 					(unit 1)
 				)
@@
 		(on_board yes)
 		(dnp no)
-		(property "Reference" "C23"
+		(property "Reference" "C49"
 			(at 144.018 69.342 0)
 			(effects
@@
 			(project "mochi_companios"
 				(path "/4ca1c142-b31d-4c3e-804c-2439f9285e87/15ca05c3-044e-4926-b1a3-d57223b2942a"
-					(reference "C23")
+					(reference "C49")
 					(unit 1)
 				)
@@
 		(dnp no)
 		(fields_autoplaced yes)
-		(property "Reference" "#PWR098"
+		(property "Reference" "#PWR0100"
 			(at 102.87 102.87 0)
 			(effects
@@
 			(project "mochi_companios"
 				(path "/4ca1c142-b31d-4c3e-804c-2439f9285e87/15ca05c3-044e-4926-b1a3-d57223b2942a"
-					(reference "#PWR098")
+					(reference "#PWR0100")
 					(unit 1)
 				)
@@
 		(on_board yes)
 		(dnp no)
-		(property "Reference" "C24"
+		(property "Reference" "C50"
 			(at 156.718 136.652 0)
 			(effects
@@
 			(project "mochi_companios"
 				(path "/4ca1c142-b31d-4c3e-804c-2439f9285e87/15ca05c3-044e-4926-b1a3-d57223b2942a"
-					(reference "C24")
+					(reference "C50")
 					(unit 1)
 				)
@@
 		(on_board yes)
 		(dnp no)
-		(property "Reference" "C64"
+		(property "Reference" "C51"
 			(at 191.008 54.102 0)
 			(effects
@@
 			(project "mochi_companios"
 				(path "/4ca1c142-b31d-4c3e-804c-2439f9285e87/15ca05c3-044e-4926-b1a3-d57223b2942a"
-					(reference "C64")
+					(reference "C51")
 					(unit 1)
 				)
@@
 		(on_board yes)
 		(dnp no)
-		(property "Reference" "R115"
+		(property "Reference" "R43"
 			(at 146.304 137.16 0)
 			(effects
@@
 			(project "mochi_companios"
 				(path "/4ca1c142-b31d-4c3e-804c-2439f9285e87/15ca05c3-044e-4926-b1a3-d57223b2942a"
-					(reference "R115")
+					(reference "R43")
 					(unit 1)
 				)
@@
 		(on_board yes)
 		(dnp no)
-		(property "Reference" "C55"
+		(property "Reference" "C47"
 			(at 95.758 104.902 0)
 			(effects
@@
 			(project "mochi_companios"
 				(path "/4ca1c142-b31d-4c3e-804c-2439f9285e87/15ca05c3-044e-4926-b1a3-d57223b2942a"
-					(reference "C55")
+					(reference "C47")
 					(unit 1)
 				)
@@
 		(dnp no)
 		(fields_autoplaced yes)
-		(property "Reference" "#PWR053"
+		(property "Reference" "#PWR0104"
 			(at 163.83 83.82 0)
 			(effects
@@
 			(project "mochi_companios"
 				(path "/4ca1c142-b31d-4c3e-804c-2439f9285e87/15ca05c3-044e-4926-b1a3-d57223b2942a"
-					(reference "#PWR053")
+					(reference "#PWR0104")
 					(unit 1)
 				)
@@
 		(on_board yes)
 		(dnp no)
-		(property "Reference" "C5"
+		(property "Reference" "C48"
 			(at 144.018 56.642 0)
 			(effects
@@
 			(project "mochi_companios"
 				(path "/4ca1c142-b31d-4c3e-804c-2439f9285e87/15ca05c3-044e-4926-b1a3-d57223b2942a"
-					(reference "C5")
+					(reference "C48")
 					(unit 1)
 				)
@@
 		(on_board yes)
 		(dnp no)
-		(property "Reference" "R46"
+		(property "Reference" "R42"
 			(at 112.014 101.6 0)
 			(effects
@@
 			(project "mochi_companios"
 				(path "/4ca1c142-b31d-4c3e-804c-2439f9285e87/15ca05c3-044e-4926-b1a3-d57223b2942a"
-					(reference "R46")
+					(reference "R42")
 					(unit 1)
 				)
@@
 		(dnp no)
 		(fields_autoplaced yes)
-		(property "Reference" "#PWR0231"
+		(property "Reference" "#PWR098"
 			(at 81.28 93.98 0)
 			(effects
@@
 			(project "mochi_companios"
 				(path "/4ca1c142-b31d-4c3e-804c-2439f9285e87/15ca05c3-044e-4926-b1a3-d57223b2942a"
-					(reference "#PWR0231")
+					(reference "#PWR098")
 					(unit 1)
 				)
@@
 		(on_board yes)
 		(dnp no)
-		(property "Reference" "#PWR047"
+		(property "Reference" "#PWR0105"
 			(at 153.67 91.44 0)
 			(effects
@@
 			(project "mochi_companios"
 				(path "/4ca1c142-b31d-4c3e-804c-2439f9285e87/15ca05c3-044e-4926-b1a3-d57223b2942a"
-					(reference "#PWR047")
+					(reference "#PWR0105")
 					(unit 1)
 				)
@@
 		(on_board yes)
 		(dnp no)
-		(property "Reference" "#PWR049"
+		(property "Reference" "#PWR0107"
 			(at 153.67 124.46 0)
 			(effects
@@
 			(project "mochi_companios"
 				(path "/4ca1c142-b31d-4c3e-804c-2439f9285e87/15ca05c3-044e-4926-b1a3-d57223b2942a"
-					(reference "#PWR049")
+					(reference "#PWR0107")
 					(unit 1)
 				)
@@
 		(on_board yes)
 		(dnp no)
-		(property "Reference" "#PWR051"
+		(property "Reference" "#PWR0111"
 			(at 198.12 66.04 0)
 			(effects
@@
 			(project "mochi_companios"
 				(path "/4ca1c142-b31d-4c3e-804c-2439f9285e87/15ca05c3-044e-4926-b1a3-d57223b2942a"
-					(reference "#PWR051")
+					(reference "#PWR0111")
 					(unit 1)
 				)
@@
 		(on_board yes)
 		(dnp no)
-		(property "Reference" "#PWR0216"
+		(property "Reference" "#PWR099"
 			(at 92.71 116.84 0)
 			(effects
@@
 			(project "mochi_companios"
 				(path "/4ca1c142-b31d-4c3e-804c-2439f9285e87/15ca05c3-044e-4926-b1a3-d57223b2942a"
-					(reference "#PWR0216")
+					(reference "#PWR099")
 					(unit 1)
 				)
@@
 		(on_board yes)
 		(dnp no)
-		(property "Reference" "#PWR050"
+		(property "Reference" "#PWR0110"
 			(at 187.96 66.04 0)
 			(effects
@@
 			(project "mochi_companios"
 				(path "/4ca1c142-b31d-4c3e-804c-2439f9285e87/15ca05c3-044e-4926-b1a3-d57223b2942a"
-					(reference "#PWR050")
+					(reference "#PWR0110")
 					(unit 1)
 				)
@@
 		(on_board yes)
 		(dnp no)
-		(property "Reference" "C66"
+		(property "Reference" "C53"
 			(at 211.328 54.102 0)
 			(effects
@@
 			(project "mochi_companios"
 				(path "/4ca1c142-b31d-4c3e-804c-2439f9285e87/15ca05c3-044e-4926-b1a3-d57223b2942a"
-					(reference "C66")
+					(reference "C53")
 					(unit 1)
 				)
@@
 		(on_board yes)
 		(dnp no)
-		(property "Reference" "#PWR052"
+		(property "Reference" "#PWR0112"
 			(at 208.28 66.04 0)
 			(effects
@@
 			(project "mochi_companios"
 				(path "/4ca1c142-b31d-4c3e-804c-2439f9285e87/15ca05c3-044e-4926-b1a3-d57223b2942a"
-					(reference "#PWR052")
+					(reference "#PWR0112")
 					(unit 1)
 				)
@@
 		(on_board yes)
 		(dnp no)
-		(property "Reference" "#PWR048"
+		(property "Reference" "#PWR0106"
 			(at 153.67 101.6 0)
 			(effects
@@
 			(project "mochi_companios"
 				(path "/4ca1c142-b31d-4c3e-804c-2439f9285e87/15ca05c3-044e-4926-b1a3-d57223b2942a"
-					(reference "#PWR048")
+					(reference "#PWR0106")
 					(unit 1)
 				)
@@
 		(on_board yes)
 		(dnp yes)
-		(property "Reference" "R47"
+		(property "Reference" "R41"
 			(at 104.394 101.6 0)
 			(effects
@@
 			(project "mochi_companios"
 				(path "/4ca1c142-b31d-4c3e-804c-2439f9285e87/15ca05c3-044e-4926-b1a3-d57223b2942a"
-					(reference "R47")
+					(reference "R41")
 					(unit 1)
 				)
@@
 		(on_board yes)
 		(dnp no)
-		(property "Reference" "#PWR097"
+		(property "Reference" "#PWR0101"
 			(at 110.49 113.03 0)
 			(effects
@@
 			(project "mochi_companios"
 				(path "/4ca1c142-b31d-4c3e-804c-2439f9285e87/15ca05c3-044e-4926-b1a3-d57223b2942a"
-					(reference "#PWR097")
+					(reference "#PWR0101")
 					(unit 1)
 				)
@@
 		(dnp no)
 		(fields_autoplaced yes)
-		(property "Reference" "#PWR03"
+		(property "Reference" "#PWR0108"
 			(at 177.8 52.07 0)
 			(effects
@@
 			(project "mochi_companios"
 				(path "/4ca1c142-b31d-4c3e-804c-2439f9285e87/15ca05c3-044e-4926-b1a3-d57223b2942a"
-					(reference "#PWR03")
+					(reference "#PWR0108")
 					(unit 1)
 				)
@@
 		(on_board yes)
 		(dnp no)
-		(property "Reference" "D4"
+		(property "Reference" "D8"
 			(at 86.36 89.408 0)
 			(effects
@@
 			(project "mochi_companios"
 				(path "/4ca1c142-b31d-4c3e-804c-2439f9285e87/15ca05c3-044e-4926-b1a3-d57223b2942a"
-					(reference "D4")
+					(reference "D8")
 					(unit 1)
 				)
@@
 		(on_board yes)
 		(dnp no)
-		(property "Reference" "#PWR0219"
+		(property "Reference" "#PWR0102"
 			(at 144.78 148.59 0)
 			(effects
@@
 			(project "mochi_companios"
 				(path "/4ca1c142-b31d-4c3e-804c-2439f9285e87/15ca05c3-044e-4926-b1a3-d57223b2942a"
-					(reference "#PWR0219")
+					(reference "#PWR0102")
 					(unit 1)
 				)
@@
 		(on_board yes)
 		(dnp no)
-		(property "Reference" "R106"
+		(property "Reference" "R40"
 			(at 86.36 98.552 90)
 			(effects
@@
 			(project "mochi_companios"
 				(path "/4ca1c142-b31d-4c3e-804c-2439f9285e87/15ca05c3-044e-4926-b1a3-d57223b2942a"
-					(reference "R106")
-					(unit 1)
-				)
+					(reference "R40")
+					(unit 1)
+				)
