File: mochi_companion/POWER.kicad_sch (KiCad schematic)
At the start: 13 parts, among them U13 TPSM82830x

Commit message: 250713_0019
Parts:
- renumbered C58 to C18, C59 to C19, C60 to C20, C61 to C21, C62 to C22, C63 to C23, D10 to D5, R40 to R14, R37 to R15, R38 to R16, R39 to R17, R36 to R18, U13 to U4
Changed lines of the file:
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@@
 		(on_board yes)
 		(dnp no)
-		(property "Reference" "#PWR0106"
+		(property "Reference" "#PWR041"
 			(at 118.11 127 0)
 			(effects
@@
 			(project "mochi_companios"
 				(path "/4ca1c142-b31d-4c3e-804c-2439f9285e87/360e48bd-6fdb-4ae5-8ff2-07b2ca7c4c87"
-					(reference "#PWR0106")
+					(reference "#PWR041")
 					(unit 1)
 				)
@@
 		(on_board yes)
 		(dnp no)
-		(property "Reference" "#PWR0110"
+		(property "Reference" "#PWR045"
 			(at 173.99 111.76 0)
 			(effects
@@
 			(project "mochi_companios"
 				(path "/4ca1c142-b31d-4c3e-804c-2439f9285e87/360e48bd-6fdb-4ae5-8ff2-07b2ca7c4c87"
-					(reference "#PWR0110")
+					(reference "#PWR045")
 					(unit 1)
 				)
@@
 		(on_board yes)
 		(dnp no)
-		(property "Reference" "#PWR0108"
+		(property "Reference" "#PWR043"
 			(at 156.21 111.76 0)
 			(effects
@@
 			(project "mochi_companios"
 				(path "/4ca1c142-b31d-4c3e-804c-2439f9285e87/360e48bd-6fdb-4ae5-8ff2-07b2ca7c4c87"
-					(reference "#PWR0108")
+					(reference "#PWR043")
 					(unit 1)
 				)
@@
 		(on_board yes)
 		(dnp no)
-		(property "Reference" "#PWR0113"
+		(property "Reference" "#PWR037"
 			(at 91.44 100.33 0)
 			(effects
@@
 			(project "mochi_companios"
 				(path "/4ca1c142-b31d-4c3e-804c-2439f9285e87/360e48bd-6fdb-4ae5-8ff2-07b2ca7c4c87"
-					(reference "#PWR0113")
+					(reference "#PWR037")
 					(unit 1)
 				)
@@
 		(on_board yes)
 		(dnp no)
-		(property "Reference" "C59"
+		(property "Reference" "C19"
 			(at 103.378 115.062 0)
 			(effects
@@
 			(project "mochi_companios"
 				(path "/4ca1c142-b31d-4c3e-804c-2439f9285e87/360e48bd-6fdb-4ae5-8ff2-07b2ca7c4c87"
-					(reference "C59")
+					(reference "C19")
 					(unit 1)
 				)
@@
 		(on_board yes)
 		(dnp no)
-		(property "Reference" "#PWR0105"
+		(property "Reference" "#PWR040"
 			(at 110.49 127 0)
 			(effects
@@
 			(project "mochi_companios"
 				(path "/4ca1c142-b31d-4c3e-804c-2439f9285e87/360e48bd-6fdb-4ae5-8ff2-07b2ca7c4c87"
-					(reference "#PWR0105")
+					(reference "#PWR040")
 					(unit 1)
 				)
@@
 		(on_board yes)
 		(dnp no)
-		(property "Reference" "R37"
+		(property "Reference" "R15"
 			(at 112.014 115.57 0)
 			(effects
@@
 			(project "mochi_companios"
 				(path "/4ca1c142-b31d-4c3e-804c-2439f9285e87/360e48bd-6fdb-4ae5-8ff2-07b2ca7c4c87"
-					(reference "R37")
+					(reference "R15")
 					(unit 1)
 				)
@@
 		(on_board yes)
 		(dnp no)
-		(property "Reference" "#PWR0107"
+		(property "Reference" "#PWR042"
 			(at 144.78 121.92 0)
 			(effects
@@
 			(project "mochi_companios"
 				(path "/4ca1c142-b31d-4c3e-804c-2439f9285e87/360e48bd-6fdb-4ae5-8ff2-07b2ca7c4c87"
-					(reference "#PWR0107")
+					(reference "#PWR042")
 					(unit 1)
 				)
@@
 		(dnp no)
 		(fields_autoplaced yes)
-		(property "Reference" "D10"
+		(property "Reference" "D5"
 			(at 208.28 109.5374 90)
 			(effects
@@
 			(project "mochi_companios"
 				(path "/4ca1c142-b31d-4c3e-804c-2439f9285e87/360e48bd-6fdb-4ae5-8ff2-07b2ca7c4c87"
-					(reference "D10")
+					(reference "D5")
 					(unit 1)
 				)
@@
 		(on_board yes)
 		(dnp no)
-		(property "Reference" "C60"
+		(property "Reference" "C20"
 			(at 159.258 99.822 0)
 			(effects
@@
 			(project "mochi_companios"
 				(path "/4ca1c142-b31d-4c3e-804c-2439f9285e87/360e48bd-6fdb-4ae5-8ff2-07b2ca7c4c87"
-					(reference "C60")
+					(reference "C20")
 					(unit 1)
 				)
@@
 		(on_board yes)
 		(dnp no)
-		(property "Reference" "C61"
+		(property "Reference" "C21"
 			(at 168.148 99.822 0)
 			(effects
@@
 			(project "mochi_companios"
 				(path "/4ca1c142-b31d-4c3e-804c-2439f9285e87/360e48bd-6fdb-4ae5-8ff2-07b2ca7c4c87"
-					(reference "C61")
+					(reference "C21")
 					(unit 1)
 				)
@@
 		(on_board yes)
 		(dnp no)
-		(property "Reference" "R39"
+		(property "Reference" "R17"
 			(at 146.304 110.49 0)
 			(effects
@@
 			(project "mochi_companios"
 				(path "/4ca1c142-b31d-4c3e-804c-2439f9285e87/360e48bd-6fdb-4ae5-8ff2-07b2ca7c4c87"
-					(reference "R39")
+					(reference "R17")
 					(unit 1)
 				)
@@
 		(dnp no)
 		(fields_autoplaced yes)
-		(property "Reference" "U13"
+		(property "Reference" "U4"
 			(at 128.905 88.9 0)
 			(effects
@@
 			(project "mochi_companios"
 				(path "/4ca1c142-b31d-4c3e-804c-2439f9285e87/360e48bd-6fdb-4ae5-8ff2-07b2ca7c4c87"
-					(reference "U13")
+					(reference "U4")
 					(unit 1)
 				)
@@
 		(on_board yes)
 		(dnp no)
-		(property "Reference" "R36"
+		(property "Reference" "R18"
 			(at 210.82 115.57 0)
 			(effects
@@
 			(project "mochi_companios"
 				(path "/4ca1c142-b31d-4c3e-804c-2439f9285e87/360e48bd-6fdb-4ae5-8ff2-07b2ca7c4c87"
-					(reference "R36")
+					(reference "R18")
 					(unit 1)
 				)
@@
 		(on_board yes)
 		(dnp no)
-		(property "Reference" "R38"
+		(property "Reference" "R16"
 			(at 146.304 100.33 0)
 			(effects
@@
 			(project "mochi_companios"
 				(path "/4ca1c142-b31d-4c3e-804c-2439f9285e87/360e48bd-6fdb-4ae5-8ff2-07b2ca7c4c87"
-					(reference "R38")
+					(reference "R16")
 					(unit 1)
 				)
@@
 		(on_board yes)
 		(dnp no)
-		(property "Reference" "C58"
+		(property "Reference" "C18"
 			(at 94.488 115.062 0)
 			(effects
@@
 			(project "mochi_companios"
 				(path "/4ca1c142-b31d-4c3e-804c-2439f9285e87/360e48bd-6fdb-4ae5-8ff2-07b2ca7c4c87"
-					(reference "C58")
+					(reference "C18")
 					(unit 1)
 				)
@@
 		(on_board yes)
 		(dnp no)
-		(property "Reference" "C62"
+		(property "Reference" "C22"
 			(at 177.038 99.822 0)
 			(effects
@@
 			(project "mochi_companios"
 				(path "/4ca1c142-b31d-4c3e-804c-2439f9285e87/360e48bd-6fdb-4ae5-8ff2-07b2ca7c4c87"
-					(reference "C62")
+					(reference "C22")
 					(unit 1)
 				)
@@
 		(on_board yes)
 		(dnp no)
-		(property "Reference" "#PWR0109"
+		(property "Reference" "#PWR044"
 			(at 165.1 111.76 0)
 			(effects
@@
 			(project "mochi_companios"
 				(path "/4ca1c142-b31d-4c3e-804c-2439f9285e87/360e48bd-6fdb-4ae5-8ff2-07b2ca7c4c87"
-					(reference "#PWR0109")
+					(reference "#PWR044")
 					(unit 1)
 				)
@@
 		(on_board yes)
 		(dnp no)
-		(property "Reference" "R40"
+		(property "Reference" "R14"
 			(at 112.014 102.87 0)
 			(effects
@@
 			(project "mochi_companios"
 				(path "/4ca1c142-b31d-4c3e-804c-2439f9285e87/360e48bd-6fdb-4ae5-8ff2-07b2ca7c4c87"
-					(reference "R40")
+					(reference "R14")
 					(unit 1)
 				)
@@
 		(on_board yes)
 		(dnp no)
-		(property "Reference" "C63"
+		(property "Reference" "C23"
 			(at 185.928 99.822 0)
 			(effects
@@
 			(project "mochi_companios"
 				(path "/4ca1c142-b31d-4c3e-804c-2439f9285e87/360e48bd-6fdb-4ae5-8ff2-07b2ca7c4c87"
-					(reference "C63")
+					(reference "C23")
 					(unit 1)
 				)
@@
 		(on_board yes)
 		(dnp no)
-		(property "Reference" "#PWR0114"
+		(property "Reference" "#PWR047"
 			(at 212.09 90.17 0)
 			(effects
@@
 			(project "mochi_companios"
 				(path "/4ca1c142-b31d-4c3e-804c-2439f9285e87/360e48bd-6fdb-4ae5-8ff2-07b2ca7c4c87"
-					(reference "#PWR0114")
+					(reference "#PWR047")
 					(unit 1)
 				)
@@
 		(on_board yes)
 		(dnp no)
-		(property "Reference" "#PWR0104"
+		(property "Reference" "#PWR039"
 			(at 100.33 127 0)
 			(effects
@@
 			(project "mochi_companios"
 				(path "/4ca1c142-b31d-4c3e-804c-2439f9285e87/360e48bd-6fdb-4ae5-8ff2-07b2ca7c4c87"
-					(reference "#PWR0104")
+					(reference "#PWR039")
 					(unit 1)
 				)
@@
 		(on_board yes)
 		(dnp no)
-		(property "Reference" "#PWR0112"
+		(property "Reference" "#PWR046"
 			(at 182.88 111.76 0)
 			(effects
@@
 			(project "mochi_companios"
 				(path "/4ca1c142-b31d-4c3e-804c-2439f9285e87/360e48bd-6fdb-4ae5-8ff2-07b2ca7c4c87"
-					(reference "#PWR0112")
+					(reference "#PWR046")
 					(unit 1)
 				)
@@
 		(on_board yes)
 		(dnp no)
-		(property "Reference" "#PWR0115"
+		(property "Reference" "#PWR048"
 			(at 212.09 127 0)
 			(effects
@@
 			(project "mochi_companios"
 				(path "/4ca1c142-b31d-4c3e-804c-2439f9285e87/360e48bd-6fdb-4ae5-8ff2-07b2ca7c4c87"
-					(reference "#PWR0115")
+					(reference "#PWR048")
 					(unit 1)
 				)
@@
 		(on_board yes)
 		(dnp no)
-		(property "Reference" "#PWR0103"
+		(property "Reference" "#PWR038"
 			(at 91.44 127 0)
 			(effects
@@
 			(project "mochi_companios"
 				(path "/4ca1c142-b31d-4c3e-804c-2439f9285e87/360e48bd-6fdb-4ae5-8ff2-07b2ca7c4c87"
-					(reference "#PWR0103")
-					(unit 1)
-				)
+					(reference "#PWR038")
+					(unit 1)
+				)
