File: mochi_companion/SD.kicad_sch (KiCad schematic)
At the start: 9 parts, among them J4 TF-018_C961679, Q2 HSST3139_C700948

Commit message: 250713_0019
Parts:
- J6: renamed from J4; footprint ESP32_C6_MINI:TF-018_C961679 -> PrjLib:0101-A-B03-006_C961679
- renumbered C26 to C54, Q2 to Q1, R43 to R44, R19 to R45, R21 to R46, R22 to R47, R20 to R48, R23 to R49
Changed lines of the file:
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@@
 		(on_board yes)
 		(dnp no)
-		(property "Reference" "#PWR054"
+		(property "Reference" "#PWR0113"
 			(at 153.67 59.69 0)
 			(effects
@@
 			(project "mochi_companios"
 				(path "/4ca1c142-b31d-4c3e-804c-2439f9285e87/f92fa38b-d1c9-454d-9780-ce8169f4308d"
-					(reference "#PWR054")
+					(reference "#PWR0113")
 					(unit 1)
 				)
@@
 		(on_board yes)
 		(dnp no)
-		(property "Reference" "J4"
+		(property "Reference" "J6"
 			(at 198.12 81.28 0)
 			(effects
@@
 			)
 		)
-		(property "Footprint" "ESP32_C6_MINI:TF-018_C961679"
+		(property "Footprint" "PrjLib:0101-A-B03-006_C961679"
 			(at 234.95 81.28 0)
 			(effects
@@
 			(project "mochi_companios"
 				(path "/4ca1c142-b31d-4c3e-804c-2439f9285e87/f92fa38b-d1c9-454d-9780-ce8169f4308d"
-					(reference "J4")
+					(reference "J6")
 					(unit 1)
 				)
@@
 		(on_board yes)
 		(dnp no)
-		(property "Reference" "#PWR057"
+		(property "Reference" "#PWR0116"
 			(at 204.47 119.38 0)
 			(effects
@@
 			(project "mochi_companios"
 				(path "/4ca1c142-b31d-4c3e-804c-2439f9285e87/f92fa38b-d1c9-454d-9780-ce8169f4308d"
-					(reference "#PWR057")
+					(reference "#PWR0116")
 					(unit 1)
 				)
@@
 		(on_board yes)
 		(dnp no)
-		(property "Reference" "R22"
+		(property "Reference" "R47"
 			(at 141.224 81.28 0)
 			(effects
@@
 			(project "mochi_companios"
 				(path "/4ca1c142-b31d-4c3e-804c-2439f9285e87/f92fa38b-d1c9-454d-9780-ce8169f4308d"
-					(reference "R22")
+					(reference "R47")
 					(unit 1)
 				)
@@
 		(on_board yes)
 		(dnp no)
-		(property "Reference" "R19"
+		(property "Reference" "R45"
 			(at 125.984 81.28 0)
 			(effects
@@
 			(project "mochi_companios"
 				(path "/4ca1c142-b31d-4c3e-804c-2439f9285e87/f92fa38b-d1c9-454d-9780-ce8169f4308d"
-					(reference "R19")
+					(reference "R45")
 					(unit 1)
 				)
@@
 		(on_board yes)
 		(dnp no)
-		(property "Reference" "R43"
+		(property "Reference" "R44"
 			(at 118.364 81.28 0)
 			(effects
@@
 			(project "mochi_companios"
 				(path "/4ca1c142-b31d-4c3e-804c-2439f9285e87/f92fa38b-d1c9-454d-9780-ce8169f4308d"
-					(reference "R43")
+					(reference "R44")
 					(unit 1)
 				)
@@
 		(on_board yes)
 		(dnp no)
-		(property "Reference" "#PWR056"
+		(property "Reference" "#PWR0115"
 			(at 153.67 101.6 0)
 			(effects
@@
 			(project "mochi_companios"
 				(path "/4ca1c142-b31d-4c3e-804c-2439f9285e87/f92fa38b-d1c9-454d-9780-ce8169f4308d"
-					(reference "#PWR056")
+					(reference "#PWR0115")
 					(unit 1)
 				)
@@
 		(on_board yes)
 		(dnp no)
-		(property "Reference" "R20"
+		(property "Reference" "R48"
 			(at 146.304 60.96 0)
 			(effects
@@
 			(project "mochi_companios"
 				(path "/4ca1c142-b31d-4c3e-804c-2439f9285e87/f92fa38b-d1c9-454d-9780-ce8169f4308d"
-					(reference "R20")
+					(reference "R48")
 					(unit 1)
 				)
@@
 		(on_board yes)
 		(dnp no)
-		(property "Reference" "R21"
+		(property "Reference" "R46"
 			(at 133.604 81.28 0)
 			(effects
@@
 			(project "mochi_companios"
 				(path "/4ca1c142-b31d-4c3e-804c-2439f9285e87/f92fa38b-d1c9-454d-9780-ce8169f4308d"
-					(reference "R21")
+					(reference "R46")
 					(unit 1)
 				)
@@
 		(on_board yes)
 		(dnp no)
-		(property "Reference" "C26"
+		(property "Reference" "C54"
 			(at 161.798 76.962 0)
 			(effects
@@
 			(project "mochi_companios"
 				(path "/4ca1c142-b31d-4c3e-804c-2439f9285e87/f92fa38b-d1c9-454d-9780-ce8169f4308d"
-					(reference "C26")
+					(reference "C54")
 					(unit 1)
 				)
@@
 		(on_board yes)
 		(dnp no)
-		(property "Reference" "Q2"
+		(property "Reference" "Q1"
 			(at 155.956 66.04 0)
 			(effects
@@
 			(project "mochi_companios"
 				(path "/4ca1c142-b31d-4c3e-804c-2439f9285e87/f92fa38b-d1c9-454d-9780-ce8169f4308d"
-					(reference "Q2")
+					(reference "Q1")
 					(unit 1)
 				)
@@
 		(on_board yes)
 		(dnp no)
-		(property "Reference" "R23"
+		(property "Reference" "R49"
 			(at 148.844 81.28 0)
 			(effects
@@
 			(project "mochi_companios"
 				(path "/4ca1c142-b31d-4c3e-804c-2439f9285e87/f92fa38b-d1c9-454d-9780-ce8169f4308d"
-					(reference "R23")
+					(reference "R49")
 					(unit 1)
 				)
@@
 		(on_board yes)
 		(dnp no)
-		(property "Reference" "#PWR055"
+		(property "Reference" "#PWR0114"
 			(at 158.75 88.9 0)
 			(effects
@@
 			(project "mochi_companios"
 				(path "/4ca1c142-b31d-4c3e-804c-2439f9285e87/f92fa38b-d1c9-454d-9780-ce8169f4308d"
-					(reference "#PWR055")
-					(unit 1)
-				)
+					(reference "#PWR0114")
+					(unit 1)
+				)
