File: mochi_companion/UART.kicad_sch (KiCad schematic)
At the start: 0 parts

Commit message: 250712_0041
Parts:
- added C18, C40, C41: 100n, Capacitor_SMD:C_0402_1005Metric, symbol Device:C
- added C39: 4u7, Capacitor_SMD:C_0402_1005Metric, symbol Device:C
- added D5: LED, Diode_SMD:D_0402_1005Metric, symbol Device:LED
- added D8: MBR0530WS, Diode_SMD:D_SOD-323, symbol Device:D_Schottky
- added R13: 330R, PCM_Resistor_SMD_AKL:R_0402_1005Metric, symbol Device:R
- added R30, R32: 5k1, PCM_Resistor_SMD_AKL:R_0402_1005Metric, symbol Device:R
- added R33, R41: 22R, PCM_Resistor_SMD_AKL:R_0402_1005Metric, symbol Device:R
- added R42, R44: 0R, PCM_Resistor_SMD_AKL:R_0402_1005Metric, symbol Device:R
- added R45: 4k7, PCM_Resistor_SMD_AKL:R_0402_1005Metric, symbol Device:R
- added U6: TYPE-C 16PIN 2MD(073)_C2765186, Connector_USB:USB_C_Receptacle_Palconn_UTC16-G, symbol ESP32_C6_MINI:USB_C_modified
- added U6: CH340E, Package_SO:MSOP-10_3x3mm_P0.5mm, symbol Interface_USB:CH340E
Connections:
- new net: D8.2 (A), U6.A4 (VBUS), U6.A9 (VBUS), U6.B4 (VBUS), U6.B9 (VBUS)
- new net: R32.1, U6.A5 (CC1)
- new net: R30.1, U6.B5 (CC2)
- new net: C18.1, R13.2, U6.S1 (SHIELD)
- new net: D5.1 (K), R45.2
- new net: D5.2 (A), U6.6 (TNOW)
- new net +3V3: C40.1, C41.1, U6.10 (V3), U6.7 (VCC)
- new net +5V: C39.1, D8.1 (K)
- new net GND: C18.2, C39.2, C40.2, C41.2, R13.1, R30.2, R32.2, R45.1, U6.3 (GND), U6.A1 (GND), U6.A12 (GND), U6.B1 (GND), U6.B12 (GND)
- new net RX: R44.2, U6.9 (RXD)
- new net RXD: R44.1
- new net TX: R42.2, U6.8 (TXD)
- new net TXD: R42.1
- new net UD_N: R33.1, U6.2 (UD-)
- new net UD_P: R41.1, U6.1 (UD+)
- new net USB_N: R33.2, U6.A7 (D-), U6.B7 (D-)
- new net USB_P: R41.2, U6.A6 (D+), U6.B6 (D+)
- no-connect marks 0 -> 4

Commit message: 250713_0019
Parts:
- renumbered C18 to C32, C39 to C33, C40 to C34, C41 to C35, D8 to D6, D5 to D7, R13 to R26, R30 to R27, R32 to R28, R33 to R29, R41 to R30, R45 to R31, R42 to R32, R44 to R33, U6 to U8, U6 to U9
Changed lines of the file:
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@@
 		(on_board yes)
 		(dnp no)
-		(property "Reference" "U6"
+		(property "Reference" "U8"
 			(at 97.79 80.01 0)
 			(effects
@@
 			(project "mochi_companios"
 				(path "/4ca1c142-b31d-4c3e-804c-2439f9285e87/725fa696-e451-457e-80b3-b9a377ed2411"
-					(reference "U6")
+					(reference "U8")
 					(unit 1)
 				)
@@
 		(on_board yes)
 		(dnp no)
-		(property "Reference" "R42"
+		(property "Reference" "R32"
 			(at 208.28 90.932 90)
 			(effects
@@
 			(project "mochi_companios"
 				(path "/4ca1c142-b31d-4c3e-804c-2439f9285e87/725fa696-e451-457e-80b3-b9a377ed2411"
-					(reference "R42")
+					(reference "R32")
 					(unit 1)
 				)
@@
 		(on_board yes)
 		(dnp no)
-		(property "Reference" "D5"
+		(property "Reference" "D7"
 			(at 193.548 123.698 90)
 			(effects
@@
 			(project "mochi_companios"
 				(path "/4ca1c142-b31d-4c3e-804c-2439f9285e87/725fa696-e451-457e-80b3-b9a377ed2411"
-					(reference "D5")
+					(reference "D7")
 					(unit 1)
 				)
@@
 		(on_board yes)
 		(dnp no)
-		(property "Reference" "#PWR093"
+		(property "Reference" "#PWR073"
 			(at 177.8 129.54 0)
 			(effects
@@
 			(project "mochi_companios"
 				(path "/4ca1c142-b31d-4c3e-804c-2439f9285e87/725fa696-e451-457e-80b3-b9a377ed2411"
-					(reference "#PWR093")
+					(reference "#PWR073")
 					(unit 1)
 				)
@@
 		(on_board yes)
 		(dnp no)
-		(property "Reference" "#PWR092"
+		(property "Reference" "#PWR072"
 			(at 165.1 95.25 0)
 			(effects
@@
 			(project "mochi_companios"
 				(path "/4ca1c142-b31d-4c3e-804c-2439f9285e87/725fa696-e451-457e-80b3-b9a377ed2411"
-					(reference "#PWR092")
+					(reference "#PWR072")
 					(unit 1)
 				)
@@
 		(on_board yes)
 		(dnp no)
-		(property "Reference" "R44"
+		(property "Reference" "R33"
 			(at 208.28 98.552 90)
 			(effects
@@
 			(project "mochi_companios"
 				(path "/4ca1c142-b31d-4c3e-804c-2439f9285e87/725fa696-e451-457e-80b3-b9a377ed2411"
-					(reference "R44")
+					(reference "R33")
 					(unit 1)
 				)
@@
 		(on_board yes)
 		(dnp no)
-		(property "Reference" "C39"
+		(property "Reference" "C33"
 			(at 142.748 55.372 0)
 			(effects
@@
 			(project "mochi_companios"
 				(path "/4ca1c142-b31d-4c3e-804c-2439f9285e87/725fa696-e451-457e-80b3-b9a377ed2411"
-					(reference "C39")
+					(reference "C33")
 					(unit 1)
 				)
@@
 		(on_board yes)
 		(dnp no)
-		(property "Reference" "#PWR084"
+		(property "Reference" "#PWR069"
 			(at 139.7 67.31 0)
 			(effects
@@
 			(project "mochi_companios"
 				(path "/4ca1c142-b31d-4c3e-804c-2439f9285e87/725fa696-e451-457e-80b3-b9a377ed2411"
-					(reference "#PWR084")
+					(reference "#PWR069")
 					(unit 1)
 				)
@@
 		(on_board yes)
 		(dnp no)
-		(property "Reference" "#PWR086"
+		(property "Reference" "#PWR070"
 			(at 154.94 82.55 0)
 			(effects
@@
 			(project "mochi_companios"
 				(path "/4ca1c142-b31d-4c3e-804c-2439f9285e87/725fa696-e451-457e-80b3-b9a377ed2411"
-					(reference "#PWR086")
+					(reference "#PWR070")
 					(unit 1)
 				)
@@
 		(on_board yes)
 		(dnp no)
-		(property "Reference" "#PWR046"
+		(property "Reference" "#PWR065"
 			(at 105.41 144.78 0)
 			(effects
@@
 			(project "mochi_companios"
 				(path "/4ca1c142-b31d-4c3e-804c-2439f9285e87/725fa696-e451-457e-80b3-b9a377ed2411"
-					(reference "#PWR046")
+					(reference "#PWR065")
 					(unit 1)
 				)
@@
 		(on_board yes)
 		(dnp no)
-		(property "Reference" "#PWR099"
+		(property "Reference" "#PWR074"
 			(at 190.5 142.24 0)
 			(effects
@@
 			(project "mochi_companios"
 				(path "/4ca1c142-b31d-4c3e-804c-2439f9285e87/725fa696-e451-457e-80b3-b9a377ed2411"
-					(reference "#PWR099")
+					(reference "#PWR074")
 					(unit 1)
 				)
@@
 		(on_board yes)
 		(dnp no)
-		(property "Reference" "#PWR090"
+		(property "Reference" "#PWR071"
 			(at 154.94 95.25 0)
 			(effects
@@
 			(project "mochi_companios"
 				(path "/4ca1c142-b31d-4c3e-804c-2439f9285e87/725fa696-e451-457e-80b3-b9a377ed2411"
-					(reference "#PWR090")
+					(reference "#PWR071")
 					(unit 1)
 				)
@@
 		(on_board yes)
 		(dnp no)
-		(property "Reference" "C18"
+		(property "Reference" "C32"
 			(at 100.838 130.302 0)
 			(effects
@@
 			(project "mochi_companios"
 				(path "/4ca1c142-b31d-4c3e-804c-2439f9285e87/725fa696-e451-457e-80b3-b9a377ed2411"
-					(reference "C18")
+					(reference "C32")
 					(unit 1)
 				)
@@
 		(on_board yes)
 		(dnp no)
-		(property "Reference" "C40"
+		(property "Reference" "C34"
 			(at 157.988 83.312 0)
 			(effects
@@
 			(project "mochi_companios"
 				(path "/4ca1c142-b31d-4c3e-804c-2439f9285e87/725fa696-e451-457e-80b3-b9a377ed2411"
-					(reference "C40")
+					(reference "C34")
 					(unit 1)
 				)
@@
 		(on_board yes)
 		(dnp no)
-		(property "Reference" "R41"
+		(property "Reference" "R30"
 			(at 134.62 102.362 90)
 			(effects
@@
 			(project "mochi_companios"
 				(path "/4ca1c142-b31d-4c3e-804c-2439f9285e87/725fa696-e451-457e-80b3-b9a377ed2411"
-					(reference "R41")
+					(reference "R30")
 					(unit 1)
 				)
@@
 		(on_board yes)
 		(dnp no)
-		(property "Reference" "R45"
+		(property "Reference" "R31"
 			(at 192.024 130.81 0)
 			(effects
@@
 			(project "mochi_companios"
 				(path "/4ca1c142-b31d-4c3e-804c-2439f9285e87/725fa696-e451-457e-80b3-b9a377ed2411"
-					(reference "R45")
+					(reference "R31")
 					(unit 1)
 				)
@@
 		(on_board yes)
 		(dnp no)
-		(property "Reference" "#PWR075"
+		(property "Reference" "#PWR066"
 			(at 124.46 129.54 0)
 			(effects
@@
 			(project "mochi_companios"
 				(path "/4ca1c142-b31d-4c3e-804c-2439f9285e87/725fa696-e451-457e-80b3-b9a377ed2411"
-					(reference "#PWR075")
+					(reference "#PWR066")
 					(unit 1)
 				)
@@
 		(on_board yes)
 		(dnp no)
-		(property "Reference" "U6"
+		(property "Reference" "U9"
 			(at 180.086 121.666 0)
 			(effects
@@
 			(project "mochi_companios"
 				(path "/4ca1c142-b31d-4c3e-804c-2439f9285e87/725fa696-e451-457e-80b3-b9a377ed2411"
-					(reference "U6")
+					(reference "U9")
 					(unit 1)
 				)
@@
 		(on_board yes)
 		(dnp no)
-		(property "Reference" "R33"
+		(property "Reference" "R29"
 			(at 134.62 94.742 90)
 			(effects
@@
 			(project "mochi_companios"
 				(path "/4ca1c142-b31d-4c3e-804c-2439f9285e87/725fa696-e451-457e-80b3-b9a377ed2411"
-					(reference "R33")
+					(reference "R29")
 					(unit 1)
 				)
@@
 		(on_board yes)
 		(dnp no)
-		(property "Reference" "#PWR076"
+		(property "Reference" "#PWR067"
 			(at 132.08 129.54 0)
 			(effects
@@
 			(project "mochi_companios"
 				(path "/4ca1c142-b31d-4c3e-804c-2439f9285e87/725fa696-e451-457e-80b3-b9a377ed2411"
-					(reference "#PWR076")
+					(reference "#PWR067")
 					(unit 1)
 				)
@@
 		(on_board yes)
 		(dnp no)
-		(property "Reference" "R13"
+		(property "Reference" "R26"
 			(at 90.424 130.81 0)
 			(effects
@@
 			(project "mochi_companios"
 				(path "/4ca1c142-b31d-4c3e-804c-2439f9285e87/725fa696-e451-457e-80b3-b9a377ed2411"
-					(reference "R13")
+					(reference "R26")
 					(unit 1)
 				)
@@
 		(on_board yes)
 		(dnp no)
-		(property "Reference" "#PWR076"
+		(property "Reference" "#PWR068"
 			(at 139.7 49.53 0)
 			(effects
@@
 			(project "mochi_companios"
 				(path "/4ca1c142-b31d-4c3e-804c-2439f9285e87/725fa696-e451-457e-80b3-b9a377ed2411"
-					(reference "#PWR076")
+					(reference "#PWR068")
 					(unit 1)
 				)
@@
 		(on_board yes)
 		(dnp no)
-		(property "Reference" "R30"
+		(property "Reference" "R27"
 			(at 127.254 118.11 0)
 			(effects
@@
 			(project "mochi_companios"
 				(path "/4ca1c142-b31d-4c3e-804c-2439f9285e87/725fa696-e451-457e-80b3-b9a377ed2411"
-					(reference "R30")
+					(reference "R27")
 					(unit 1)
 				)
@@
 		(on_board yes)
 		(dnp no)
-		(property "Reference" "R32"
+		(property "Reference" "R28"
 			(at 134.874 118.11 0)
 			(effects
@@
 			(project "mochi_companios"
 				(path "/4ca1c142-b31d-4c3e-804c-2439f9285e87/725fa696-e451-457e-80b3-b9a377ed2411"
-					(reference "R32")
+					(reference "R28")
 					(unit 1)
 				)
@@
 		(on_board yes)
 		(dnp no)
-		(property "Reference" "#PWR045"
+		(property "Reference" "#PWR064"
 			(at 97.79 144.78 0)
 			(effects
@@
 			(project "mochi_companios"
 				(path "/4ca1c142-b31d-4c3e-804c-2439f9285e87/725fa696-e451-457e-80b3-b9a377ed2411"
-					(reference "#PWR045")
+					(reference "#PWR064")
 					(unit 1)
 				)
@@
 		(on_board yes)
 		(dnp no)
-		(property "Reference" "C41"
+		(property "Reference" "C35"
 			(at 168.148 83.312 0)
 			(effects
@@
 			(project "mochi_companios"
 				(path "/4ca1c142-b31d-4c3e-804c-2439f9285e87/725fa696-e451-457e-80b3-b9a377ed2411"
-					(reference "C41")
+					(reference "C35")
 					(unit 1)
 				)
@@
 		(on_board yes)
 		(dnp no)
-		(property "Reference" "D8"
+		(property "Reference" "D6"
 			(at 129.286 46.99 0)
 			(effects
@@
 			(project "mochi_companios"
 				(path "/4ca1c142-b31d-4c3e-804c-2439f9285e87/725fa696-e451-457e-80b3-b9a377ed2411"
-					(reference "D8")
-					(unit 1)
-				)
+					(reference "D6")
+					(unit 1)
+				)
