File: mochi_companion/mochi_companios.kicad_sch (KiCad schematic)
At the start: 28 parts, among them J1 USB_C_Receptacle_USB2.0_16P, J2 Conn_01x04_MountingPin, SW1 SW_Push, SW2 SW_Push, U1 ESP32-C6-MINI-1/U, Y1 32768Hz

Commit message: 250712_0041
Parts:
- removed C11: 100n, Capacitor_SMD:C_0402_1005Metric, symbol Device:C
- removed C4: 4u7, Capacitor_SMD:C_0402_1005Metric, symbol Device:C
- removed C8: 1u, Capacitor_SMD:C_0402_1005Metric, symbol Device:C
- removed R9: 22R, Resistor_SMD:R_0402_1005Metric, symbol Device:R
- removed SW1, SW2: SW_Push, Button_Switch_SMD:SW_Push_SPST_NO_Alps_SKRK, symbol Switch:SW_Push
- added C25: 100n, Capacitor_SMD:C_0402_1005Metric, symbol Device:C
- added C30, C37: 4u7, Capacitor_SMD:C_0402_1005Metric, symbol Device:C
- added R26: 330R, PCM_Resistor_SMD_AKL:R_0402_1005Metric, symbol Device:R
- added SW2, SW3: 1TS026A-2300-0553-CT, PrjLib:1TS026A-2300-0553-CT, symbol Switch:SW_MEC_5E
- C1, C3: Field5 (none) -> C0402; Field6 (none) -> 50V
- C2: value 100n -> 1u; Field5 (none) -> C0402; Field6 (none) -> 25V
- C6: Field5 (none) -> C0402; Field6 (none) -> 16V
- C7: value 4u7 -> 100n; Field5 (none) -> C0402; Field6 (none) -> 50V
- D3: Field5 (none) -> D0402
- R2: value 330R -> 5k1; footprint Resistor_SMD:R_0402_1005Metric -> PCM_Resistor_SMD_AKL:R_0402_1005Metric; Field5 (none) -> R0402
- R3, R6, R8: footprint Resistor_SMD:R_0402_1005Metric -> PCM_Resistor_SMD_AKL:R_0402_1005Metric; Field5 (none) -> R0402
- R4: value 5k1 -> 4k7; footprint Resistor_SMD:R_0402_1005Metric -> PCM_Resistor_SMD_AKL:R_0402_1005Metric; Field5 (none) -> R0402
- R5: value 4k7 -> 10k; footprint Resistor_SMD:R_0402_1005Metric -> PCM_Resistor_SMD_AKL:R_0402_1005Metric; Field5 (none) -> R0402
- R7: value 10k -> 22R; footprint Resistor_SMD:R_0402_1005Metric -> PCM_Resistor_SMD_AKL:R_0402_1005Metric; Field5 (none) -> R0402
Connections:
- net BUSY is gone; now on net MOSI: U1.24 (IO18)
- net D/C is gone; now on net SDA: U1.26 (IO20)
- net RST is gone; now on net CS: U1.25 (IO19)
- net +3V3: now also R5.2, R6.2, C30.1; no longer R6.1, R7.1
- net +5V: now also C37.1
- net CS: no longer U1.5 (IO2)
- net D_N: now also R7.2; no longer R8.1
- net D_P: now also R8.2
- net GND: now also R2.1, R3.1, R4.1, C25.2, C30.2, C37.2, R26.1, SW2.1, SW2.2, SW3.1, SW3.2; no longer R2.2, R3.2, R4.2, R5.2
- net I2C_EN: now also U1.29 (IO23); no longer U1.9 (IO4)
- net MOSI: no longer U1.6 (IO3)
- net PC1: now also SW2.3 (K), SW2.4 (A)
- net SCK: now also U1.27 (IO21); no longer U1.16 (IO7)
- net SDA: no longer U1.15 (IO6)
- net USB_N: now also R7.1; no longer R8.2
- net USB_P: now also R8.1
- net at J1.A5 (CC1): now also R2.2; no longer R3.1
- net at C2.1, U1.8 (EN): now also C3.1, R5.1, SW3.3 (K), SW3.4 (A); no longer R7.2
- net CLK: now reaches U1.19 (IO14)
- net MISO: now reaches U1.20 (IO15)
- net at U1.22 (IO8): now also R6.1; no longer R6.2
- net SD_EN: now reaches U1.28 (IO22)
- net at J1.B5 (CC2): now also R3.2; no longer R4.1
- net at D3.1 (K): now also R4.2; no longer R5.1
- net SCLK renamed DATA_IN
- new net: C25.1, J1.S1 (SHIELD), R26.2
- new net BCLK: U1.5 (IO2)
- new net DATA_OUT: U1.9 (IO4)
- new net GPS_RX: U1.16 (IO7)
- new net GPS_TX: U1.15 (IO6)
- new net LRCLK: U1.6 (IO3)
Other:
- added sheet OLED (OLED.kicad_sch)
- added sheet SD (SD.kicad_sch)
- sheet AUDIO ports: added DATA_IN, DATA_OUT; removed DAC_DATA, DAC_DIN, DAC_SD
- sheet GPS ports: added RX, TX; removed none
- moved on the sheet: J2

Commit message: 250713_0019
Parts:
- added R50: 0R, PCM_Resistor_SMD_AKL:R_0402_1005Metric, symbol Device:R
- U1: footprint prj_footprint:ESP32-C6-MINI-1 -> RF_Module:ESP32-C6-MINI-1
- renumbered C25 to C1, C13 to C10, C37 to C2, C1 to C4, C2 to C5, C30 to C6, C6 to C7, C7 to C8, C12 to C9, D11 to D1, D3 to D2, R26 to R1, R11 to R10, R6 to R5, R5 to R6, R10 to R9, SW3 to SW1
Connections:
- net X0: now also R50.1
- new net AUDIO/GAIN: R50.2
Other:
- sheet AUDIO ports: added GAIN; removed none
